Commit message: new file:   .gitignore 	modified:   description/realsense.xacro 	modified:   ignition/astro.urdf 	modified:   ignition/proba.urdf

File: description/realsense.xacro (robot description, xacro)
@@ -99,4 +99,5 @@
     </joint>
     <link name="camera_color_frame"/>
+    <!-- Komentar -->
     <joint name="camera_color_optical_joint" type="fixed">
       <origin xyz="0 0 0" rpy="${-M_PI/2} 0 ${-M_PI/2}" />

File: ignition/astro.urdf (robot description, URDF)
Before this commit: robot astro, 9 links, 8 joints
Links:
- removed link base_footprint
- removed link base_link
Joints:
- removed joint base_link_joint
- removed joint chasis_joint

File: ignition/proba.urdf (robot description, URDF)
Before this commit: robot astro, 9 links, 8 joints
Links:
- added link depth_camera_link; visual mesh 
Joints:
- added joint front_depth_camera_joint: type fixed, parent , child 
